File: kicad/remote.kicad_pcb (KiCad board)
At the start: 2 copper layers, 31.8 x 55.9 mm, 23 parts, among them J1 ICSP, SW0 EVQ-Q2K02W, SW1 EVQ-Q2K02W, SW2 EVQ-Q2K02W, U1 ATtiny85-20S, U2 Ai-Thinker NF-03

Commit message: Update PCB to fit mechanism 1. Change back side battery holder GND pad connection to solid 2. Chnage 'ICSP' to 'ISP' 3. Move ISP header 4. Increase ISP VDD track width 5. Made ISP harder to "Pogo" style
Parts:
- J1: moved to B.Cu
- moved J1 10.5 mm to (28.6, 31.1), turned to 180 degrees
- moved R3 1.81 mm to (22.1, 31.0)
- moved R2 1.59 mm to (22.1, 33.1)
- moved RN1 1.55 mm to (21.3, 27.7)
- renumbered R3* to R3
Routing:
- net Net-(J1-Pad5): track 3.76 -> 16.9 mm, vias 1 -> 2
- net Net-(J1-Pad3): track 5.30 -> 14.3 mm, vias 1 -> 2
- net Net-(J1-Pad2): track 8.60 -> 14.6 mm, vias 1 -> 2
- net Net-(J1-Pad1): track 6.74 -> 10.8 mm, vias 1 -> 2
- net /SW1: track 39.5 -> 37.6 mm, vias 5 -> 6
- net /DO: track 17.5 -> 18.9 mm
- net /DI: track 20.0 -> 21.3 mm
- net /SCK: track 16.4 -> 17.5 mm
- net Net-(BT1-Pad1): track 92.7 -> 91.6 mm
- net /RST: track 33.6 -> 32.8 mm
- net Net-(J1-Pad4): track 9.76 -> 10.3 mm, vias 1 -> 2
- net GND: vias 87 -> 80
Other:
- board text added: "City Science Lab @ Taipei Tech DANCHOUZHOU 2022-11-10"
- board text added: "ISP"
- board text removed: "City Science Lab @ Taipei Tech DANCHOUZHOU 2022-11-07"
- board text removed: "ICSP"
